Commit message: Gripper orientation and multiple gripper loading

File: objects/Nestle_Nips_Hard_Candy_Peanut_Butter/Nestle_Nips_Hard_Candy_Peanut_Butter.urdf (robot description, URDF)
Before this commit: robot Nestle_Nips_Hard_Candy_Peanut_Butter, 1 links, 0 joints
Links:
- link baseLink: geometry collision mesh filename=./meshes/model.obj scale=1.0 1.0 1.0; visual mesh filename=./meshes/model.obj scale=1.0 1.0 1.0
