Commit message: feat: updated hithand urdf and usd

File: grippers/hithand/hithand.urdf (robot description, URDF)
Before this commit: robot hithand, 23 links, 22 joints
Links:
- link Right_Index_Phaprox: geometry collision mesh filename=./meshes/collision/finger/hit-hand-2-finger-phaprox-cropped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; visual mesh filename=./meshes/visual/finger/hit-hand-2-finger-phaprox.obj
- link Right_Little_Phaprox: geometry collision mesh filename=./meshes/collision/finger/hit-hand-2-finger-phaprox-cropped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; visual mesh filename=./meshes/visual/finger/hit-hand-2-finger-phaprox.obj
- link Right_Thumb_Phaprox: geometry collision mesh filename=./meshes/collision/finger/hit-hand-2-finger-phaprox-cropped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; visual mesh filename=./meshes/visual/finger/hit-hand-2-finger-phaprox.obj
- link base_link_hithand: geometry collision mesh filename=./meshes/collision/palm/hit-hand-2-palm-right-merged_faces_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; visual mesh filename=./meshes/visual/palm/hit-hand-2-palm-right.obj

Commit message: fix: updated base link pose for hithand

File: grippers/hithand/hithand.urdf (robot description, URDF)
Before this commit: robot hithand, 23 links, 22 joints
Joints:
- joint fixed: origin xyz=0 0 0.1 rpy=0 0 0 -> xyz=0 0 0 rpy=0 0 0

File: grippers/hithand/hithand_.urdf (robot description, URDF)
Before this commit: robot hithand, 23 links, 22 joints
Joints:
- joint fixed: origin xyz=0 0 0.1 rpy=0 0 0 -> xyz=0 0 0 rpy=0 0 0
